File: sch_and_pcb/kicad_fingers_spi.sch (KiCad schematic (older format))
At the start: 40 parts, among them J1 RJ45, J2 RJ45, J3 8PIN_CONN, J4 8PIN_CONN, J5 8PIN_CONN, J6 8PIN_CONN, J7 8PIN_CONN, J8 8PIN_CONN, P1 CONN_01X03, P2 CONN_01X03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

Commit message: Fixed an issue where the secondary spi addresses could block the bus.
Parts:
- added U4: 74LS126, symbol 74LS126
- renumbered U4 to U5
Connections:
- net GND: now also U4.7 (GND), U4.7 (GND), U4.7 (GND), U4.7 (GND)
- net SS1-A: now also U4.1 (E), U4.10 (E), U4.13 (E), U4.4 (E)
- net SS3-A: now also U4.2, U4.3
- net SS4-A: now also U4.5 (D), U4.6 (O)
- net SS5-A: now also U4.8, U4.9 (D)
- net SS6-A: now also U4.11, U4.12
- net VCC: now also U4.14 (VCC), U4.14 (VCC), U4.14 (VCC), U4.14 (VCC)
Other:
- note added: "74HC126"
- note added: "An additional buffer gate to be able to\ndeselect the secundary SPI devices\nwith SS1-A"
- moved on the sheet: J7, J8, RR2
